Commit message: Added Camera

File: src/rita_description/urdf/rita.urdf (robot description, URDF)
Before this commit: robot RITA, 6 links, 5 joints
Joints:
- joint link_4_Rigid-4: origin xyz=0.10794414999999997 0.0 -0.0197 rpy=-3.141592653589793 -1.5707963267948966 0 -> xyz=0.10794414999999997 0.0 -0.0197 rpy=-3.141592653589793 0 0

Commit message: fixed end-effector

File: src/rita_description/urdf/rita.urdf (robot description, URDF)
Before this commit: robot RITA, 6 links, 5 joints
Joints:
- joint base_Revolute-1: limit lower=-3.14159 upper=3.14159 effort=2.94 velocity=11.1 -> lower=-3 upper=3 effort=2.94 velocity=11.1
- joint link_2_Revolute-2: limit lower=-3.14159 upper=3.14159 effort=1.47 velocity=11.1 -> lower=-1.57 upper=1.57 effort=1.47 velocity=11.1
- joint link_3_Revolute-3: limit lower=-3.14159 upper=3.14159 effort=2.94 velocity=11.1 -> lower=-2.09 upper=2.09 effort=2.94 velocity=11.1

Commit message: created Yolo streaming package

File: src/rita_description/urdf/rita.urdf (robot description, URDF)
Before this commit: robot RITA, 6 links, 5 joints
Joints:
- joint link_4_Rigid-4: origin xyz=0.10794414999999997 0.0 -0.0197 rpy=-3.141592653589793 0 0 -> xyz=0.10794414999999997 0.0 -0.0197 rpy=-3.141592653589793 -1.5707963267948966 0

File: src/rita_moveit2_config/config/RITA.ros2_control.xacro (robot description, xacro)
@@ -1,50 +1,79 @@
 <?xml version="1.0"?>
 <robot xmlns:xacro="http://www.ros.org/wiki/xacro">
-    <xacro:macro name="RITA_ros2_control" params="name initial_positions_file">
+    <xacro:macro name="RITA_ros2_control" params="name initial_positions_file use_gazebo:=false">
         <xacro:property name="initial_positions" value="${xacro.load_yaml(initial_positions_file)['initial_positions']}"/>
-        <ros2_control name="${name}" type="system">
-            <hardware>
-                <plugin>waveshare_servos/WaveshareServos</plugin>
-            </hardware>
-            <joint name="base_Revolute-1">
-                <param name="id">3</param>
-                <param name="type">pos</param>
-                <param name="offset">3.14159265</param>
-                <param name="direction">-1.0</param>
-                <command_interface name="position"/>
-                <state_interface name="position">
-                  <param name="initial_value">${initial_positions['base_Revolute-1']}</param>
-                </state_interface>
-                <state_interface name="velocity"/>
-                <state_interface name="torque"/>
-                <state_interface name="temperature"/>
-            </joint>
-            <joint name="link_2_Revolute-2">
-                <param name="id">2</param>
-                <param name="type">pos</param>
-                <param name="offset">3.14159265</param>
-                <param name="direction">-1.0</param>
-                <command_interface name="position"/>
-                <state_interface name="position">
-                  <param name="initial_value">${initial_positions['link_2_Revolute-2']}</param>
-                </state_interface>
-                <state_interface name="velocity"/>
-                <state_interface name="torque"/>
-                <state_interface name="temperature"/>
-            </joint>
-            <joint name="link_3_Revolute-3">
-                <param name="id">1</param>
-                <param name="type">pos</param>
-                <param name="offset">3.14159265</param>
-                <param name="direction">-1.0</param>
-                <command_interface name="position"/>
-                <state_interface name="position">
-                  <param name="initial_value">${initial_positions['link_3_Revolute-3']}</param>
-                </state_interface>
-                <state_interface name="velocity"/>
-                <state_interface name="torque"/>
-                <state_interface name="temperature"/>
-            </joint>
-        </ros2_control>
+        <xacro:if value="${use_gazebo}">
+            <ros2_control name="GazeboSimSystem" type="system">
+                <hardware>
+                    <plugin>gz_ros2_control/GazeboSimSystem</plugin>
+                </hardware>
+                <joint name="base_Revolute-1">
+                    <command_interface name="position"/>
+                    <state_interface name="position"/>
+                    <state_interface name="velocity"/>
+                </joint>
+                <joint name="link_2_Revolute-2">
+                    <command_interface name="position"/>
+                    <state_interface name="position"/>
+                    <state_interface name="velocity"/>
+                </joint>
+                <joint name="link_3_Revolute-3">
+                    <command_interface name="position"/>
+                    <state_interface name="position"/>
+                    <state_interface name="velocity"/>
+                </joint>
+            </ros2_control>
+            <gazebo>
+                <plugin filename="gz_ros2_control-system" name="gz_ros2_control::GazeboSimROS2ControlPlugin">
+                    <parameters>$(find rita_gazebo)/config/ros2_controllers.yaml</parameters>
+                </plugin>
+            </gazebo>
+        </xacro:if>
+        <xacro:unless value="${use_gazebo}">
+            <ros2_control name="${name}" type="system">
+                <hardware>
+                    <plugin>waveshare_servos/WaveshareServos</plugin>
+                </hardware>
+                <joint name="base_Revolute-1">
+                    <param name="id">3</param>
+                    <param name="type">pos</param>
+                    <param name="offset">3.14159265</param>
+                    <param name="direction">-1.0</param>
+                    <command_interface name="position"/>
+                    <state_interface name="position">
+                      <param name="initial_value">${initial_positions['base_Revolute-1']}</param>
+                    </state_interface>
+                    <state_interface name="velocity"/>
+                    <state_interface name="torque"/>
+                    <state_interface name="temperature"/>
+                </joint>
+                <joint name="link_2_Revolute-2">
+                    <param name="id">2</param>
+                    <param name="type">pos</param>
+                    <param name="offset">3.14159265</param>
+                    <param name="direction">-1.0</param>
+                    <command_interface name="position"/>
+                    <state_interface name="position">
+                      <param name="initial_value">${initial_positions['link_2_Revolute-2']}</param>
+                    </state_interface>
+                    <state_interface name="velocity"/>
+                    <state_interface name="torque"/>
+                    <state_interface name="temperature"/>
+                </joint>
+                <joint name="link_3_Revolute-3">
+                    <param name="id">1</param>
+                    <param name="type">pos</param>
+                    <param name="offset">3.14159265</param>
+                    <param name="direction">-1.0</param>
+                    <command_interface name="position"/>
+                    <state_interface name="position">
+                      <param name="initial_value">${initial_positions['link_3_Revolute-3']}</param>
+                    </state_interface>
+                    <state_interface name="velocity"/>
+                    <state_interface name="torque"/>
+                    <state_interface name="temperature"/>
+                </joint>
+            </ros2_control>
+        </xacro:unless>
     </xacro:macro>
 </robot>

File: src/rita_moveit2_config/config/RITA.urdf.xacro (robot description, xacro)
@@ -2,8 +2,7 @@
 <robot xmlns:xacro="http://www.ros.org/wiki/xacro" name="RITA">
     <xacro:arg name="initial_positions_file" default="initial_positions.yaml" />
-    <!-- Import RITA urdf file -->
+    <xacro:arg name="use_gazebo" default="false" />
     <xacro:include filename="$(find rita_description)/urdf/rita.urdf" />
-    <!-- Import control_xacro -->
     <xacro:include filename="RITA.ros2_control.xacro" />
-    <xacro:RITA_ros2_control name="FakeSystem" initial_positions_file="$(arg initial_positions_file)"/>
+    <xacro:RITA_ros2_control name="FakeSystem" initial_positions_file="$(arg initial_positions_file)" use_gazebo="$(arg use_gazebo)"/>
 </robot>
